File: kicad/main_board/main_board/main_board.kicad_sch (KiCad schematic)
At the start: 14 parts, among them U1 AMS1117, U2 Pico, U3 NRF24L01_Breakout, U4 TXS0108EPW

Commit message: [feat]final versions of boards + gerbers
Parts:
- added C1, C10, C5, C6, C7, C8: 1uf, Capacitor_SMD:C_0805_2012Metric, symbol Device:C
- added C9: 10uf, Capacitor_SMD:CP_Elec_6.3x5.4, symbol Device:C
- added D1, D2: D, Diode_SMD:D_1206_3216Metric, symbol Device:D
- added H1, H2, H3, H4: MountingHole, MountingHole:MountingHole_3mm, symbol Mechanical:MountingHole
- added R1, R2: R, Resistor_SMD:R_1206_3216Metric, symbol Device:R
- added R3: 10k, Resistor_SMD:R_1206_3216Metric, symbol Device:R
- added SW1, SW2, SW3: SW_Push, Button_Switch_THT:SW_PUSH_6mm, symbol Switch:SW_Push
- added U5: AMS1117, Package_TO_SOT_SMD:SOT-223-3_TabPin2, symbol Regulator_Linear:AMS1117
- C2: renamed from C3; footprint (none) -> Capacitor_SMD:CP_Elec_6.3x5.4
- U4: renamed from U2; footprint RPi_Pico:RPi_Pico_SMD_TH -> pi:RPi_Pico_SMD_TH
- renumbered BT2 to BT1, BT1 to BT2, C2 to C3, C1 to C4, U4 to U2
Connections:
- net 3.3V+: now also C10.2, C6.1, R2.1
- net 5V+: now also C1.1, C7.1, R1.1, U5.2 (VO)
- net BAT+: now also C5.1, C8.1, C9.1, U5.3 (VI)
- net GND: now also C1.2, C10.1, C5.2, C6.2, C7.2, C8.2, C9.2, D1.1 (K), D2.1 (K), R3.1, SW1.2, SW2.2, SW3.2, U5.1 (ADJ)
- net LED_1: now also U4.9 (GPIO6); no longer U4.5 (GPIO3)
- net LED_2: now also U4.10 (GPIO7); no longer U4.7 (GPIO5)
- net LED_3: now also U4.11 (GPIO8); no longer U4.10 (GPIO7)
- net PWM_1_3v3: now also U2.5 (A4); no longer U2.1 (A1)
- net PWM_2_3v3: now also U2.4 (A3), U4.5 (GPIO3); no longer U2.3 (A2), U4.6 (GPIO4)
- net PWM_3_3v3: now also U2.3 (A2), U4.6 (GPIO4); no longer U2.4 (A3), U4.9 (GPIO6)
- net PWM_4_3v3: now also U2.1 (A1), U4.7 (GPIO5); no longer U2.5 (A4), U4.11 (GPIO8)
- net RX: now also U2.15 (B5); no longer U2.14 (B6)
- net RX_3.3: now also U2.6 (A5); no longer U2.7 (A6)
- net TX: now also U2.14 (B6); no longer U2.15 (B5)
- net TX_3.3: now also U2.7 (A6); no longer U2.6 (A5)
- net at U2.10 (OE): now also R3.2
- net TEST_1: now reaches U4.19 (GPIO14)
- net TEST_1: now also SW1.1
- net TEST_2: now reaches U4.20 (GPIO15)
- net TEST_2: now also SW2.1
- net TEST_3: now reaches U4.26 (GPIO20)
- net TEST_3: now also SW3.1
- new net: D1.2 (A), R1.2
- new net: D2.2 (A), R2.2
- no-connect marks 5 -> 16
Other:
- note added: "DC DC CONVERTER"
- note added: "POWER LEDS"
- note added: "TEST BUTTONS"
- moved on the sheet: U2, U4
