File: kicad/servo_plate/servo_plate.kicad_pcb (KiCad board)
At the start: 2 copper layers, 66.5 x 31.5 mm, 8 parts, among them J1 Conn_01x05_Pin, M1 Motor_Servo, SW1 SW_Push

Commit message: [feat]final versions of boards + gerbers
Parts:
- added C2: 1uf, Capacitor_SMD:C_0805_2012Metric, F.Cu at (146.8, 79.5)
- J1: footprint Connector_JST:JST_PH_B5B-PH-K_1x05_P2.00mm_Vertical -> TerminalBlock_TE-Connectivity:TerminalBlock_TE_282834-5_1x05_P2.54mm_Horizontal
- moved J1 3.75 mm to (86.2, 69.5)
Connections:
- J1 pad 5: SW1 -> BUTTON
Routing:
- net BUTTON: track 0.00 -> 82.1 mm
- net SW1: track 57.3 -> 0.00 mm
- net GND: track 3.61 -> 23.8 mm, vias 1 -> 18
- net 5V+: track 41.3 -> 48.9 mm
- net PWM: track 78.3 -> 82.0 mm
- net LED: track 44.4 -> 48.0 mm
- net BAT+: track 8.83 -> 11.6 mm
