File: kicad/servo_plate/servo_plate.kicad_sch (KiCad schematic)
At the start: 8 parts, among them J1 Conn_01x05_Pin, M1 Motor_Servo, SW1 SW_Push

Commit message: [feat]final versions of boards + gerbers
Parts:
- added C2: 1uf, Capacitor_SMD:C_0805_2012Metric, symbol Device:C
- J1: footprint Connector_JST:JST_PH_B5B-PH-K_1x05_P2.00mm_Vertical -> TerminalBlock_TE-Connectivity:TerminalBlock_TE_282834-5_1x05_P2.54mm_Horizontal
Connections:
- net SW1 is gone; now on net BUTTON: J1.5 (Pin_5)
- net 5V+: now also C2.2
- net GND: now also C2.1
Changed lines of the file:
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@@
 	(paper "A4")
+	(junction
+		(at 153.67 82.55)
+		(diameter 0)
+		(color 0 0 0 0)
+	)
 	(junction
 		(at 184.15 110.49)
@@
 	)
 	(junction
+		(at 153.67 74.93)
+		(diameter 0)
+		(color 0 0 0 0)
+	)
+	(junction
 		(at 189.23 52.07)
 		(diameter 0)
@@
 	(wire
 		(pts
-			(xy 149.86 76.2) (xy 160.02 76.2)
+			(xy 149.86 74.93) (xy 153.67 74.93)
 		)
 		(stroke
@@
 	(wire
 		(pts
+			(xy 163.83 81.28) (xy 163.83 82.55)
+		)
+		(stroke
+			(width 0)
+			(type default)
+		)
+	)
+	(wire
+		(pts
 			(xy 179.07 110.49) (xy 184.15 110.49)
 		)
@@
 	(wire
 		(pts
+			(xy 153.67 82.55) (xy 148.59 82.55)
+		)
+		(stroke
+			(width 0)
+			(type default)
+		)
+	)
+	(wire
+		(pts
+			(xy 161.29 74.93) (xy 161.29 76.2)
+		)
+		(stroke
+			(width 0)
+			(type default)
+		)
+	)
+	(wire
+		(pts
 			(xy 139.7 111.76) (xy 148.59 111.76)
 		)
@@
 	(wire
 		(pts
+			(xy 153.67 74.93) (xy 161.29 74.93)
+		)
+		(stroke
+			(width 0)
+			(type default)
+		)
+	)
+	(wire
+		(pts
 			(xy 190.5 113.03) (xy 190.5 115.57)
 		)
@@
 	(wire
 		(pts
-			(xy 148.59 82.55) (xy 154.94 82.55)
+			(xy 163.83 82.55) (xy 153.67 82.55)
+		)
+		(stroke
+			(width 0)
+			(type default)
+		)
+	)
+	(wire
+		(pts
+			(xy 163.83 81.28) (xy 165.1 81.28)
 		)
 		(stroke
@@
 	(wire
 		(pts
-			(xy 149.86 76.2) (xy 149.86 80.01)
+			(xy 149.86 74.93) (xy 149.86 80.01)
 		)
 		(stroke
@@
 		)
 	)
-	(global_label "SW1"
+	(global_label "BUTTON"
 		(shape input)
 		(at 179.07 120.65 0)
@@
 		)
 		(property "Intersheetrefs" "${INTERSHEET_REFS}"
-			(at 185.9256 120.65 0)
+			(at 189.2519 120.65 0)
 			(effects
 				(font
@@
 				(justify left)
 				(hide yes)
+			)
+		)
+	)
+	(symbol
+		(lib_id "Device:C")
+		(at 153.67 78.74 0)
+		(unit 1)
+		(exclude_from_sim no)
+		(in_bom yes)
+		(on_board yes)
+		(dnp no)
+		(fields_autoplaced yes)
+		(property "Reference" "C2"
+			(at 157.48 77.4699 0)
+			(effects
+				(font
+					(size 1.27 1.27)
+				)
+				(justify left)
+			)
+		)
+		(property "Value" "1uf"
+			(at 157.48 80.0099 0)
+			(effects
+				(font
+					(size 1.27 1.27)
+				)
+				(justify left)
+			)
+		)
+		(property "Footprint" "Capacitor_SMD:C_0805_2012Metric"
+			(at 154.6352 82.55 0)
+			(effects
+				(font
+					(size 1.27 1.27)
+				)
+				(hide yes)
+			)
+		)
+		(property "Datasheet" "~"
+			(at 153.67 78.74 0)
+			(effects
+				(font
+					(size 1.27 1.27)
+				)
+				(hide yes)
+			)
+		)
+		(property "Description" "Unpolarized capacitor"
+			(at 153.67 78.74 0)
+			(effects
+				(font
+					(size 1.27 1.27)
+				)
+				(hide yes)
+			)
+		)
+		(pin "2"
+		)
+		(pin "1"
+		)
+		(instances
+			(project ""
+				(path "/5e15e14e-53de-4d47-aff7-4d61b34e8085"
+					(reference "C2")
+					(unit 1)
+				)
 			)
 		)
@@
 	(symbol
 		(lib_id "power:GND")
-		(at 160.02 76.2 0)
+		(at 161.29 76.2 0)
 		(unit 1)
 		(exclude_from_sim no)
@@
 		(fields_autoplaced yes)
 		(property "Reference" "#PWR04"
-			(at 160.02 82.55 0)
+			(at 161.29 82.55 0)
 			(effects
 				(font
@@
 		)
 		(property "Value" "GND"
-			(at 160.02 81.28 0)
+			(at 161.29 81.28 0)
 			(effects
 				(font
@@
 		)
 		(property "Footprint" ""
-			(at 160.02 76.2 0)
+			(at 161.29 76.2 0)
 			(effects
 				(font
@@
 		)
 		(property "Datasheet" ""
-			(at 160.02 76.2 0)
+			(at 161.29 76.2 0)
 			(effects
 				(font
@@
 		)
 		(property "Description" "Power symbol creates a global label with name \"GND\" , ground"
-			(at 160.02 76.2 0)
+			(at 161.29 76.2 0)
 			(effects
 				(font
@@
 	(symbol
 		(lib_id "power:VBUS")
-		(at 154.94 82.55 0)
+		(at 165.1 81.28 0)
 		(unit 1)
 		(exclude_from_sim no)
@@
 		(dnp no)
 		(property "Reference" "#PWR06"
-			(at 154.94 86.36 0)
+			(at 165.1 85.09 0)
 			(effects
 				(font
@@
 		)
 		(property "Value" "5V+"
-			(at 154.94 78.486 0)
+			(at 165.1 77.216 0)
 			(effects
 				(font
@@
 		)
 		(property "Footprint" ""
-			(at 154.94 82.55 0)
+			(at 165.1 81.28 0)
 			(effects
 				(font
@@
 		)
 		(property "Datasheet" ""
-			(at 154.94 82.55 0)
+			(at 165.1 81.28 0)
 			(effects
 				(font
@@
 		)
 		(property "Description" "Power symbol creates a global label with name \"VBUS\""
-			(at 154.94 82.55 0)
+			(at 165.1 81.28 0)
 			(effects
 				(font
@@
 			)
 		)
-		(property "Footprint" "Connector_JST:JST_PH_B5B-PH-K_1x05_P2.00mm_Vertical"
+		(property "Footprint" "TerminalBlock_TE-Connectivity:TerminalBlock_TE_282834-5_1x05_P2.54mm_Horizontal"
 			(at 173.99 115.57 0)
 			(effects
